File: pcb/cardo.kicad_pcb (KiCad board)
At the start: 2 copper layers, 256.8 x 95.3 mm, 55 parts, among them J1 Conn_01x02_Pin, SW1 SW_Push, SW10 SW_Push, SW11 SW_Push, SW12 SW_Push, SW13 SW_Push, SW14 SW_Push, SW15 SW_Push, SW16 SW_Push, SW17 SW_Push, SW18 SW_Push, SW19 SW_Push, SW2 SW_Push, SW20 SW_Push, SW21 SW_Push, SW22 SW_Push, SW23 SW_Push, SW24 SW_Push, SW25 SW_Push, SW26 SW_Push, SW27 SW_Push, SW28 SW_Push, SW29 SW_Push, SW3 SW_Push, SW30 SW_Push, SW31 SW_Push, SW32 SW_Push, SW33 SW_Push, SW34 SW_Push, SW35 SW_Push, SW36 SW_Push, SW37 SW_Push, SW38 RotaryEncoder, SW39 RotaryEncoder, SW4 SW_Push, SW5 SW_Push, SW6 SW_Push, SW7 SW_Push, SW8 SW_Push, SW9 SW_Push, U1 74HC595, U2 74HC595, U3 74HC595, U4 MODULE_102010448, U5 74HC595, U6 74HC595

Commit message: Update hardware files for SN74HCS596
Parts:
- U1, U2, U3, U5, U6: value 74HC595 -> SN74HCS596DR
Changed lines of the file:
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@@
 			)
 		)
-		(property "Value" "74HC595"
+		(property "Value" "SN74HCS596DR"
 			(at 0 5.9 100)
 			(layer "F.Fab")
@@
 			)
 		)
-		(property "Datasheet" "http://www.ti.com/lit/ds/symlink/sn74hc595.pdf"
+		(property "Datasheet" "https://www.ti.com/lit/ds/symlink/sn74hcs596.pdf"
 			(at 0 0 100)
 			(layer "F.Fab")
@@
 			)
 		)
-		(property "Description" "8-bit serial in/out Shift Register 3-State Outputs"
+		(property "Description" "Texas Instruments 8-bit shift register with Schmitt-trigger inputs and open-drain outputs"
 			(at 0 0 100)
 			(layer "F.Fab")
@@
 			)
 		)
-		(property "Value" "74HC595"
+		(property "Value" "SN74HCS596DR"
 			(at 0 5.899999 100)
 			(layer "F.Fab")
@@
 			)
 		)
-		(property "Datasheet" "http://www.ti.com/lit/ds/symlink/sn74hc595.pdf"
+		(property "Datasheet" "https://www.ti.com/lit/ds/symlink/sn74hcs596.pdf"
 			(at 0 0 100)
 			(layer "F.Fab")
@@
 			)
 		)
-		(property "Description" "8-bit serial in/out Shift Register 3-State Outputs"
+		(property "Description" "Texas Instruments 8-bit shift register with Schmitt-trigger inputs and open-drain outputs"
 			(at 0 0 100)
 			(layer "F.Fab")
@@
 			)
 		)
-		(property "Value" "74HC595"
+		(property "Value" "SN74HCS596DR"
 			(at 0 5.9 80)
 			(layer "F.Fab")
@@
 			)
 		)
-		(property "Datasheet" "http://www.ti.com/lit/ds/symlink/sn74hc595.pdf"
+		(property "Datasheet" "https://www.ti.com/lit/ds/symlink/sn74hcs596.pdf"
 			(at 0 0 80)
 			(layer "F.Fab")
@@
 			)
 		)
-		(property "Description" "8-bit serial in/out Shift Register 3-State Outputs"
+		(property "Description" "Texas Instruments 8-bit shift register with Schmitt-trigger inputs and open-drain outputs"
 			(at 0 0 80)
 			(layer "F.Fab")
@@
 			)
 		)
-		(property "Value" "74HC595"
+		(property "Value" "SN74HCS596DR"
 			(at 0 5.9 80)
 			(layer "F.Fab")
@@
 			)
 		)
-		(property "Datasheet" "http://www.ti.com/lit/ds/symlink/sn74hc595.pdf"
+		(property "Datasheet" "https://www.ti.com/lit/ds/symlink/sn74hcs596.pdf"
 			(at 0 0 80)
 			(layer "F.Fab")
@@
 			)
 		)
-		(property "Description" "8-bit serial in/out Shift Register 3-State Outputs"
+		(property "Description" "Texas Instruments 8-bit shift register with Schmitt-trigger inputs and open-drain outputs"
 			(at 0 0 80)
 			(layer "F.Fab")
@@
 			)
 		)
-		(property "Value" "74HC595"
+		(property "Value" "SN74HCS596DR"
 			(at 0 5.9 90)
 			(layer "F.Fab")
@@
 			)
 		)
-		(property "Datasheet" "http://www.ti.com/lit/ds/symlink/sn74hc595.pdf"
+		(property "Datasheet" "https://www.ti.com/lit/ds/symlink/sn74hcs596.pdf"
 			(at 0 0 90)
 			(layer "F.Fab")
@@
 			)
 		)
-		(property "Description" "8-bit serial in/out Shift Register 3-State Outputs"
+		(property "Description" "Texas Instruments 8-bit shift register with Schmitt-trigger inputs and open-drain outputs"
 			(at 0 0 90)
 			(layer "F.Fab")
